File: RCboat.kicad_sch (KiCad schematic)
At the start: 60 parts, among them J1 Battery, J3 Conn_02x10_Odd_Even, M1 Motor_Servo, M2 Motor_Servo, SW1 SW_Push_Dual, SW2 SW_Push_SPDT, U1 STM32F100C4Tx, U2 BD9G341EFJ, U33 AMS1117-3.3, U4 MPU-6000, Y1 8.000MHZ

Commit message: Add files via upload
recent files of the schemes
Parts:
- removed C1, C3, C4: 20p, Capacitor_THT:CP_Axial_L10.0mm_D4.5mm_P15.00mm_Horizontal, symbol pspice:CAP
- removed C14, C330, C331: 10u, symbol pspice:C
- removed C15: 0.1u, symbol pspice:C
- removed C16, C_RC_1, C_RC_2: 100u, symbol pspice:C
- removed C2, C7: 10uF, Capacitor_THT:CP_Axial_L10.0mm_D4.5mm_P15.00mm_Horizontal, symbol Device:C
- removed C5, C6: 100nF, symbol Device:C
- removed C8: 1uF, Capacitor_THT:CP_Axial_L10.0mm_D4.5mm_P15.00mm_Horizontal, symbol Device:C
- removed C9: 0.1u, symbol Device:C
- removed C?: 6800p, symbol pspice:C
- removed C_RC_3: 1.5p, symbol pspice:C
- removed C_RC_4: 1.0p, symbol pspice:C
- removed C_RC_5, C_RC_6: 22p, symbol pspice:C
- removed C_RC_7: 10n, symbol pspice:C
- removed C_RC_8: 1n, symbol pspice:C
- removed C_RC_9: 33n, symbol pspice:C
- removed J1: Battery, Battery:BatteryHolder_Bulgin_BX0036_1xC, symbol Connector_Generic:Conn_01x02
- removed J3: Conn_02x10_Odd_Even, symbol Connector_Generic:Conn_02x10_Odd_Even
- removed L_RC_1: 2.7n, symbol pspice:INDUCTOR
- removed L_RC_2: 8.2n, symbol pspice:INDUCTOR
- removed L_RC_3: 3.9n, symbol pspice:INDUCTOR
- removed R12, R13, R?: 10k, symbol Device:R
- removed R14: 10K, symbol Device:R
- removed R15: 390, symbol Device:R
- removed R_RC_1: 1M, symbol Device:R
- removed R_RC_2: 22K, symbol Device:R
- removed U1: STM32F100C4Tx, Package_QFP:LQFP-48_7x7mm_P0.5mm, symbol MCU_ST_STM32F1:STM32F100C4Tx
- removed U2: BD9G341EFJ, Package_SO:HTSOP-8-1EP_3.9x4.9mm_P1.27mm_EP2.4x3.2mm_ThermalVias, symbol Regulator_Switching:BD9G341EFJ
- removed U33: AMS1117-3.3, Package_TO_SOT_SMD:SOT-223-3_TabPin2, symbol Regulator_Linear:AMS1117-3.3
- removed U4: MPU-6000, Sensor_Motion:InvenSense_QFN-24_4x4mm_P0.5mm, symbol Sensor_Motion:MPU-6000
- removed U?: NRF24L01_Breakout, RF_Module:nRF24L01_Breakout, symbol RF:NRF24L01_Breakout
- removed U_RC: NRF24L01, Package_DFN_QFN:QFN-20-1EP_4x4mm_P0.5mm_EP2.5x2.5mm, symbol RF:NRF24L01
- removed Y_RC: Crystal, symbol Device:Crystal
- added C1, C2, C3: 10u, Capacitor_SMD:C_1210_3225Metric_Pad1.33x2.70mm_HandSolder, symbol pspice:C
- added C13: 10uF, Capacitor_SMD:C_1210_3225Metric_Pad1.33x2.70mm_HandSolder, symbol Device:C
- added C14: 1uF, Capacitor_SMD:C_1210_3225Metric_Pad1.33x2.70mm_HandSolder, symbol Device:C
- added C15, C16: 100nF, Capacitor_SMD:C_1210_3225Metric_Pad1.33x2.70mm_HandSolder, symbol Device:C
- added C17: 0.1u, Capacitor_SMD:C_1210_3225Metric_Pad1.33x2.70mm_HandSolder, symbol Device:C
- added C18: 2.2u, Capacitor_SMD:C_1210_3225Metric_Pad1.33x2.70mm_HandSolder, symbol Device:C
- added C4: 0.1u, Capacitor_SMD:C_1210_3225Metric_Pad1.33x2.70mm_HandSolder, symbol pspice:C
- added C5: 6800p, Capacitor_SMD:C_1210_3225Metric_Pad1.33x2.70mm_HandSolder, symbol pspice:C
- added C6, C7, C8: 20p, Capacitor_SMD:C_1210_3225Metric_Pad1.33x2.70mm_HandSolder, symbol pspice:CAP
- added C9: 100u, Capacitor_SMD:C_1210_3225Metric_Pad1.33x2.70mm_HandSolder, symbol pspice:C
- added J1: Conn_02x10_Odd_Even, symbol Connector_Generic:Conn_02x10_Odd_Even
- added J2: Battery, Battery:BatteryHolder_Bulgin_BX0036_1xC, symbol Connector_Generic:Conn_01x02
- added R10: 0.75k, Resistor_SMD:R_0603_1608Metric_Pad0.98x0.95mm_HandSolder, symbol Device:R
- added R6, R7: 10k, Resistor_SMD:R_0603_1608Metric_Pad0.98x0.95mm_HandSolder, symbol Device:R
- added R8: 10K, Resistor_SMD:R_0603_1608Metric_Pad0.98x0.95mm_HandSolder, symbol Device:R
- added R9: 3k, Resistor_SMD:R_0603_1608Metric_Pad0.98x0.95mm_HandSolder, symbol Device:R
- added U1: BD9G341EFJ, Package_SO:HTSOP-8-1EP_3.9x4.9mm_P1.27mm_EP2.4x3.2mm_ThermalVias, symbol Regulator_Switching:BD9G341EFJ
- added U2: AMS1117-3.3, Package_TO_SOT_SMD:SOT-223-3_TabPin2, symbol Regulator_Linear:AMS1117-3.3
- added U3: NRF24L01_Breakout, RF_Module:nRF24L01_Breakout, symbol RF:NRF24L01_Breakout
- added U4: STM32F100C4Tx, Package_QFP:LQFP-48_7x7mm_P0.5mm, symbol MCU_ST_STM32F1:STM32F100C4Tx
- added U5: MPU-6000, Sensor_Motion:InvenSense_QFN-24_4x4mm_P0.5mm, symbol Sensor_Motion:MPU-6000
- C10: value 2.2u -> 10uF; footprint (none) -> Capacitor_SMD:C_1210_3225Metric_Pad1.33x2.70mm_HandSolder
- C11, C12: footprint (none) -> Capacitor_SMD:C_1210_3225Metric_Pad1.33x2.70mm_HandSolder
- D1: footprint (none) -> Diode_SMD:D_0201_0603Metric_Pad0.64x0.40mm_HandSolder
- L1: footprint (none) -> Inductor_SMD:L_0603_1608Metric_Pad1.05x0.95mm_HandSolder
- R1: value R -> 100k; footprint (none) -> Resistor_SMD:R_0603_1608Metric_Pad0.98x0.95mm_HandSolder
- R11: value 10k -> 390; footprint (none) -> Resistor_SMD:R_0603_1608Metric_Pad0.98x0.95mm_HandSolder
- R2: value R -> 20k; footprint (none) -> Resistor_SMD:R_0603_1608Metric_Pad0.98x0.95mm_HandSolder
- R3: value 47k -> 10k; footprint (none) -> Resistor_SMD:R_0603_1608Metric_Pad0.98x0.95mm_HandSolder
- R4: value 3k -> 10k; footprint (none) -> Resistor_SMD:R_0603_1608Metric_Pad0.98x0.95mm_HandSolder
- R5: value 0.75k -> 47k; footprint (none) -> Resistor_SMD:R_0603_1608Metric_Pad0.98x0.95mm_HandSolder
- Y1: footprint (none) -> Crystal:Crystal_SMD_0603-2Pin_6.0x3.5mm_HandSoldering
Connections:
- net +BATT: now also C1.1, J2.1 (Pin_1), U1.8 (VCC)
- net 5V: now also C2.1, C9.1, R9.1, U2.3 (VI); no longer R4.1
- net GND: now also C1.2, C13.2, C14.2, C15.2, C16.2, C17.2, C18.2, C2.2, C3.2, C6.2, C7.2, C8.1, C9.2, J1.10 (Pin_10), J1.12 (Pin_12), J1.14 (Pin_14), J1.16 (Pin_16), J1.18 (Pin_18), J1.20 (Pin_20), J1.4 (Pin_4), J1.6 (Pin_6), J1.8 (Pin_8), J2.2 (Pin_2), R10.1, R10.2, R6.2, R7.2, R9.2, U1.2 (GND), U1.4 (FB), U2.1 (GND), U3.1 (GND), U4.23 (VSS), U4.35 (VSS), U4.47 (VSS), U4.8 (VSSA), U5.1 (CLKIN), U5.11 (FSYNC), U5.18 (GND); no longer R11.2, R5.1
- net JTDI: now also J1.5 (Pin_5), U4.38 (PA15)
- net OSC_IN: now also C6.1, U4.5 (PD0)
- net OSC_OUT: now also R11.1, U4.6 (PD1)
- net SPI1_CS: now also U3.4 (~{CSN}), U4.14 (PA4), U5.8 (~{CS})
- net SPI1_MISO: now also U3.7 (MISO), U4.16 (PA6), U5.9 (AD0/MISO)
- net SPI1_MOSI: now also U3.6 (MOSI), U4.17 (PA7), U5.24 (SDA/MOSI)
- net SPI1_SCK: now also U3.5 (SCK), U4.15 (PA5), U5.23 (SCL/SCLK)
- net SPI2_MOSI: now also U4.28 (PB15), U5.6 (AUX_SDA)
- net SPI2_SCK: now also U4.26 (PB13), U5.7 (AUX_SCL)
- net SWCLK: now also J1.9 (Pin_9), U4.37 (PA14)
- net SWDIO: now also J1.7 (Pin_7), U4.34 (PA13)
- net TDO: now also J1.13 (Pin_13), U4.39 (PB3)
- net TIM1_CH1: now also U4.29 (PA8)
- net TIM1_CH2: now also U4.30 (PA9)
- net TIM1_CH3: now also U4.31 (PA10)
- net VDD: now also C10.1, C13.1, C14.1, C15.1, C16.1, C3.1, J1.1 (Pin_1), J1.2 (Pin_2), U2.2 (VO), U3.2 (VCC), U4.1 (VBAT), U4.24 (VDD), U4.36 (VDD), U4.48 (VDD), U4.9 (VDDA), U5.13 (VDD)
- net at D1.1 (K), L1.1: now also C4.2, U1.1 (LX)
- net at R3.1: now also J1.11 (Pin_11)
- net at R1.2, R2.1: now also U1.6 (EN)
- net at SW1.2, SW1.4: now also C8.2, J1.15 (Pin_15), U4.7 (NRST)
- net at Y1.2: now also R11.2, C7.1
- net at SW2.2 (B): now also R8.2
- new net: R8.1, U4.44 (BOOT0)
- new net: J1.19 (Pin_19), R6.1
- new net: C4.1, U1.7 (BST)
- new net: C17.1, U5.10 (REGOUT)
- new net: C5.1, U1.3 (VC)
- new net: C5.2, R7.1
- new net: J1.17 (Pin_17), R4.1
- new net: J1.3 (Pin_3), U4.40 (PB4)
- new net: R5.1, U1.5 (RT)
- new net: C18.1, U5.20 (CPOUT)
- no-connect marks 7 -> 24
Other:
- note removed: "Probably not correct but i will leave it here for now"
- company: Z. Nyamanza  -> (none)
- title: RC Boat -> (none)

Commit message: Add files via upload
Parts:
- added J3: Conn_01x02, Connector_AMASS:AMASS_XT30U-F_1x02_P5.0mm_Vertical, symbol Connector_Generic:Conn_01x02
- J1: footprint (none) -> Connector_PinSocket_2.54mm:PinSocket_2x10_P2.54mm_Vertical
- J2: footprint Battery:BatteryHolder_Bulgin_BX0036_1xC -> Connector_AMASS:AMASS_XT30U-F_1x02_P5.0mm_Vertical
- SW1, SW2: footprint (none) -> Button_Switch_SMD:SW_Push_SPST_NO_Alps_SKRK
Connections:
- net +BATT: now also J3.1 (Pin_1)
- net 5V: no longer BLDC1.2 (Pin_2)
- net GND: now also J3.2 (Pin_2)
- no-connect marks 24 -> 25
Other:
- note added: "Connectors"
- note added: "Power Subsystem"
- moved on the sheet: BLDC1, C1, C10, C11, C12, C13, C14, C15, C16, C17, C18, C2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

Commit message: Add files via upload
Parts:
- removed SW1: SW_Push_Dual, Button_Switch_SMD:SW_Push_SPST_NO_Alps_SKRK, symbol Switch:SW_Push_Dual
- removed SW2: SW_Push_SPDT, Button_Switch_SMD:SW_Push_SPST_NO_Alps_SKRK, symbol Switch:SW_Push_SPDT
- added SW1: SW_Push, Button_Switch_THT:SW_PUSH_6mm, symbol Switch:SW_Push
- added SW2: SW_SPDT, Button_Switch_THT:SW_Slide_1P2T_CK_OS102011MS2Q, symbol Switch:SW_SPDT
- C1, C10, C11, C12, C13, C14, C15, C16, C17, C18, C2, C3, C4, C5, C6, C7, C8, C9: footprint Capacitor_SMD:C_1210_3225Metric_Pad1.33x2.70mm_HandSolder -> Capacitor_SMD:C_0603_1608Metric_Pad1.08x0.95mm_HandSolder
- D1: footprint Diode_SMD:D_0201_0603Metric_Pad0.64x0.40mm_HandSolder -> Diode_SMD:D_1206_3216Metric_Pad1.42x1.75mm_HandSolder
- J1: footprint Connector_PinSocket_2.54mm:PinSocket_2x10_P2.54mm_Vertical -> Connector_PinHeader_2.54mm:PinHeader_2x10_P2.54mm_Vertical
- J3: value Conn_01x02 -> Battery
Connections:
- net +BATT: now also SW2.3 (C); no longer J2.1 (Pin_1), J3.1 (Pin_1)
- net GND: now also R8.2, SW1.1; no longer D1.2 (A), R10.1, R9.2, U1.4 (FB)
- net at C8.2, J1.15 (Pin_15), U4.7 (NRST): now also SW1.2
- new net: J2.1 (Pin_1), J3.1 (Pin_1), SW2.2 (B)
- new net: D1.2 (A), R10.1, R9.2, U1.4 (FB)
- no-connect marks 25 -> 26
Other:
- note added: "BLDC/Servo1/Servo2"
- note added: "Power"
- note removed: "Connectors"
- note removed: "Power Subsystem"
- moved on the sheet: BLDC1, C1, C10, C11, C12, C13, C14, C15, C16, C17, C18, C2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
