File: Final 1.0/RCboat.kicad_pcb (KiCad board)
At the start: 2 copper layers, 45.5 x 50 mm, 45 parts, among them J1 Conn_02x10_Odd_Even, J2 Battery, J3 Battery, M1 Motor_Servo, M2 Motor_Servo, SW1 SW_Push, SW2 SW_SPDT, U1 BD9G341EFJ, U2 AMS1117-3.3, U3 NRF24L01_Breakout, U4 STM32F100C4Tx, U5 MPU-6000, Y1 8.000MHZ

Commit message: Add files via upload
Parts:
- added REF: MountingHole_2.1mm, MountingHole:MountingHole_2.1mm, F.Cu at (158.8, 105.3)
- added REF: MountingHole_2.1mm, MountingHole:MountingHole_2.1mm, F.Cu at (118.9, 82.8)
- added REF: MountingHole_2.1mm, MountingHole:MountingHole_2.1mm, F.Cu at (118.9, 127.2)
- moved J2 3.87 mm to (121.6, 114.9)
- moved J3 3.87 mm to (121.6, 107.7)
- moved SW2 3.87 mm to (122.1, 122.2)
Changed lines of the file:
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@@
   )
   (footprint "Connector_AMASS:AMASS_XT30U-F_1x02_P5.0mm_Vertical" (layer "F.Cu")
-    (at 120.9 118.7025)
+    (at 121.6 114.9)
     (descr "Connector XT30 Vertical Cable Female, https://www.tme.eu/en/Document/3cbfa5cfa544d79584972dd5234a409e/XT30U%20SPEC.pdf")
     (tags "RC Connector XT30")
@@
       (rotate (xyz 0 0 0))
     )
+  )
+  (footprint "MountingHole:MountingHole_2.1mm" (layer "F.Cu")
+    (at 158.8 105.3 90)
+    (descr "Mounting Hole 2.1mm, no annular")
+    (tags "mounting hole 2.1mm no annular")
+    (attr exclude_from_pos_files exclude_from_bom)
+    (fp_text reference "REF" (at 0 -1.7 90) (layer "F.SilkS")
+      (effects (font (size 1 1) (thickness 0.15)))
+    )
+    (fp_text value "MountingHole_2.1mm" (at 0 3.2 90) (layer "F.Fab")
+      (effects (font (size 1 1) (thickness 0.15)))
+    )
+    (fp_text user "${REFERENCE}" (at 0 0 90) (layer "F.Fab")
+      (effects (font (size 1 1) (thickness 0.15)))
+    )
+    (fp_circle (center 0 0) (end 2.1 0) (layer "Cmts.User") (width 0.15) (fill none))
+    (fp_circle (center 0 0) (end 2.35 0) (layer "F.CrtYd") (width 0.05) (fill none))
+    (pad "" np_thru_hole circle (at 0 0 90) (size 2.1 2.1) (drill 2.1) (layers *.Cu *.Mask))
   )
   (footprint "Resistor_SMD:R_0603_1608Metric_Pad0.98x0.95mm_HandSolder" (layer "F.Cu")
@@
     )
   )
+  (footprint "MountingHole:MountingHole_2.1mm" (layer "F.Cu")
+    (at 118.9 82.8)
+    (descr "Mounting Hole 2.1mm, no annular")
+    (tags "mounting hole 2.1mm no annular")
+    (attr exclude_from_pos_files exclude_from_bom)
+    (fp_text reference "REF" (at 0.4 -1.7) (layer "F.SilkS")
+      (effects (font (size 1 1) (thickness 0.15)))
+    )
+    (fp_text value "MountingHole_2.1mm" (at 0 3.2) (layer "F.Fab")
+      (effects (font (size 1 1) (thickness 0.15)))
+    )
+    (fp_text user "${REFERENCE}" (at 0 0) (layer "F.Fab")
+      (effects (font (size 1 1) (thickness 0.15)))
+    )
+    (fp_circle (center 0 0) (end 2.1 0) (layer "Cmts.User") (width 0.15) (fill none))
+    (fp_circle (center 0 0) (end 2.35 0) (layer "F.CrtYd") (width 0.05) (fill none))
+    (pad "" np_thru_hole circle (at 0 0) (size 2.1 2.1) (drill 2.1) (layers *.Cu *.Mask))
+  )
   (footprint "Capacitor_SMD:C_0603_1608Metric_Pad1.08x0.95mm_HandSolder" (layer "F.Cu")
     (at 142 118)
@@
       (rotate (xyz 0 0 0))
     )
+  )
+  (footprint "MountingHole:MountingHole_2.1mm" (layer "F.Cu")
+    (at 118.9 127.2 90)
+    (descr "Mounting Hole 2.1mm, no annular")
+    (tags "mounting hole 2.1mm no annular")
+    (attr exclude_from_pos_files exclude_from_bom)
+    (fp_text reference "REF" (at 0 -1.8 90) (layer "F.SilkS")
+      (effects (font (size 1 1) (thickness 0.15)))
+    )
+    (fp_text value "MountingHole_2.1mm" (at 0 3.2 90) (layer "F.Fab")
+      (effects (font (size 1 1) (thickness 0.15)))
+    )
+    (fp_text user "${REFERENCE}" (at 0 0 90) (layer "F.Fab")
+      (effects (font (size 1 1) (thickness 0.15)))
+    )
+    (fp_circle (center 0 0) (end 2.1 0) (layer "Cmts.User") (width 0.15) (fill none))
+    (fp_circle (center 0 0) (end 2.35 0) (layer "F.CrtYd") (width 0.05) (fill none))
+    (pad "" np_thru_hole circle (at 0 0 90) (size 2.1 2.1) (drill 2.1) (layers F&B.Cu *.Mask))
   )
   (footprint "Package_QFP:LQFP-48_7x7mm_P0.5mm" (layer "F.Cu")
@@
   )
   (footprint "Connector_AMASS:AMASS_XT30U-F_1x02_P5.0mm_Vertical" (layer "F.Cu")
-    (at 120.9 111.5)
+    (at 121.6 107.6975)
     (descr "Connector XT30 Vertical Cable Female, https://www.tme.eu/en/Document/3cbfa5cfa544d79584972dd5234a409e/XT30U%20SPEC.pdf")
     (tags "RC Connector XT30")
@@
   )
   (footprint "Button_Switch_THT:SW_Slide_1P2T_CK_OS102011MS2Q" (layer "F.Cu")
-    (at 121.4 126)
+    (at 122.1 122.1975)
     (descr "CuK miniature slide switch, OS series, SPDT, https://www.ckswitches.com/media/1428/os.pdf")
     (tags "switch SPDT")
@@
   (segment (start 147.14 116.241072) (end 147.14 112.44) (width 0.2) (layer "B.Cu") (net 3))
   (segment (start 148.499464 117.600536) (end 147.14 116.241072) (width 0.2) (layer "B.Cu") (net 3))
-  (segment (start 125.4 126) (end 125.4 127.6) (width 0.6) (layer "F.Cu") (net 4))
-  (segment (start 125.4 127.6) (end 126.5 128.7) (width 0.6) (layer "F.Cu") (net 4))
-  (segment (start 133.7375 128.7) (end 136.2375 126.2) (width 0.6) (layer "F.Cu") (net 4))
+  (segment (start 129.52125 127.46875) (end 134.96875 127.46875) (width 0.6) (layer "F.Cu") (net 4))
+  (segment (start 134.96875 127.46875) (end 136.2375 126.2) (width 0.6) (layer "F.Cu") (net 4))
   (segment (start 137.85 124.405) (end 136.795 124.405) (width 0.4) (layer "F.Cu") (net 4))
   (segment (start 137.845 124.4) (end 137.85 124.405) (width 0.4) (layer "F.Cu") (net 4))
@@
   (segment (start 135.5125 124.4) (end 137.845 124.4) (width 0.4) (layer "F.Cu") (net 4))
   (segment (start 136.795 124.405) (end 136.2375 124.9625) (width 0.4) (layer "F.Cu") (net 4))
-  (segment (start 126.5 128.7) (end 133.7375 128.7) (width 0.6) (layer "F.Cu") (net 4))
+  (segment (start 126.1 122.1975) (end 126.1 124.0475) (width 0.6) (layer "F.Cu") (net 4))
+  (segment (start 126.1 124.0475) (end 129.52125 127.46875) (width 0.6) (layer "F.Cu") (net 4))
   (segment (start 143.185 102.6625) (end 143.185 104.1225) (width 0.2) (layer "F.Cu") (net 5))
   (segment (start 139.7 90.415) (end 139.7 91.6) (width 0.2) (layer "F.Cu") (net 5))
@@
   (segment (start 141 104) (end 141.185 103.815) (width 0.2) (layer "F.Cu") (net 60))
   (segment (start 141.185 103.815) (end 141.185 102.6625) (width 0.2) (layer "F.Cu") (net 60))
-  (segment (start 120.9 111.5) (end 120.9 118.7025) (width 1) (layer "F.Cu") (net 61))
-  (segment (start 123.4 121.2025) (end 123.4 126) (width 1) (layer "F.Cu") (net 61))
-  (segment (start 120.9 118.7025) (end 123.4 121.2025) (width 1) (layer "F.Cu") (net 61))
+  (segment (start 121.6 107.6975) (end 121.6 114.9) (width 1) (layer "F.Cu") (net 61))
+  (segment (start 124.1 117.4) (end 124.1 122.1975) (width 1) (layer "F.Cu") (net 61))
+  (segment (start 121.6 114.9) (end 124.1 117.4) (width 1) (layer "F.Cu") (net 61))
   (zone (net 3) (net_name "GND") (layer "F.Cu") (hatch edge 0.508)
     (connect_pads (clearance 0.2))
